Commit message: detection done

File: urdf/robot.urdf.xacro (robot description, xacro)
@@ -1,34 +1,37 @@
 <?xml version="1.0"?>
-<robot xmlns:xacro="http://www.ros.org/wiki/xacro">
-  <xacro:property name="pi" value="3.1415926535897931" />
-  <!-- This first link called "world" is empty -->
-  <link name="world"></link>
-  <!-- A simple fixed joint from our empty world link, to our base. -->
-  <!-- The base origin is offset from the world origin. -->
-  <joint name="base_joint" type="fixed">
-    <origin xyz="2 2 0" rpy="0 0 0"/>
-    <parent link="world"/>
-    <child link="base_link"/>
-  </joint>
-  <link name="base_link">
-    <visual>
-      <origin xyz="0 0 0" rpy="0 0 0"/>
-      <geometry>
-        <box size="1 1 1" />
-      </geometry>
-      <material name="blue">
-        <color rgba="0 0 1 1"/>
-      </material>
-    </visual>
-    <collision>
-      <origin xyz="0 0 0" rpy="0 0 0"/>
-      <geometry>
-        <box size="1 1 1" />
-      </geometry>
-    </collision>
-    <inertial>
-      <origin xyz="0 0 0" rpy="0 0 0"/>
-      <mass value="1" />
-    </inertial>
-  </link>
+<robot name="robot_name" xmlns:xacro="http://www.ros.org/wiki/xacro">
+    <xacro:arg name="color" default="Blue"/>
+    <xacro:arg name="x" default="0.0"/>
+    <xacro:arg name="y" default="0.0"/>
+    <xacro:arg name="z" default="0.0"/>
+    <xacro:property name="pi" value="3.1415926535897931" />
+    <xacro:property name="color" value="$(arg color)"/>
+    <xacro:property name="x" value="$(arg x)"/>
+    <xacro:property name="y" value="$(arg y)"/>
+    <xacro:property name="z" value="$(arg z)"/>
+    <xacro:property name="d" value="0.4"/>
+    <xacro:property name="l" value="0.4"/>
+    <xacro:property name="h" value="0.4"/>
+    <link name="my_box">
+        <inertial>
+            <origin xyz="${x} ${y} ${z}"/>
+            <mass value="1.0" />
+            <inertia  ixx="1.0" ixy="0.0"  ixz="0.0"  iyy="100.0"  iyz="0.0"  izz="1.0" />
+        </inertial>
+        <visual>
+            <origin xyz="${x} ${y} ${z+h/2}"/>
+            <geometry>
+                <box size="${d} ${l} ${h}" />
+            </geometry>
+        </visual>
+        <collision>
+            <origin xyz="${x} ${y} ${z+h/2}"/>
+            <geometry>
+                <box size="${d} ${l} ${h}" />
+            </geometry>
+        </collision>
+    </link>
+    <gazebo reference="my_box">
+        <material>Gazebo/${color}</material>
+    </gazebo>
 </robot>
